File: 2026_C_AV_LPSU/2026_C_AV_LPSU.kicad_pcb (KiCad board)
At the start: 4 copper layers, 80 x 80 mm, 120 parts, among them IC1 LTC4090EDJC#PBF, IC2 LT3960EMSE#PBF, IC3 LTC3425EUH#PBF, IC4 TPS7A0533PDBZR, IC5 LTC4368IMS-1#PBF, J1 DIN41612_02x16_AB, Q1 FDS9926A, Q3 PSMN6R4-30MLDX, U1 SI2333DS-T1-E3, U2 SI2333DS-T1-E3, U3 INA228, U4 INA228, U6 LTC4357DCB

Commit message: LPSU & TMB
Parts:
- removed the G*** at (165.6, 71.2)
- removed the G*** at (135.9, 119.0)
- removed the G*** at (123.0, 118.9)
- removed the G*** at (153.8, 114.5)
- added ?: , clipboard:c18867c1-0f3b-4b99-910a-bd5b356c13f5, F.Cu at (143.0, 88.3)
- added D13: BLUE, LED_SMD:LED_0603_1608Metric, F.Cu at (136.3, 140.9)
- added D14: SBRT5A50SAF-13, SBRT5A50SAF-13:SODFL5226X110N, F.Cu at (112.6, 88.1)
- added F1: Polyfuse, 2016L260_24MR:2016L26024MR, F.Cu at (106.8, 91.2)
- added G***: LOGO, LOGO, F.Cu at (166.0, 71.5)
- added G***: LOGO, LOGO, B.Cu at (153.8, 114.5)
- added G***: LOGO, LOGO, B.Cu at (160.4, 139.1)
- added J2: Conn_01x03_Pin, Connector_PinHeader_2.54mm:PinHeader_1x03_P2.54mm_Vertical_SMD_Pin1Right, F.Cu at (164.3, 139.2)
- added J3: Conn_01x02_Pin, TerminalBlock_Phoenix:TerminalBlock_Phoenix_PT-1,5-2-3.5-H_1x02_P3.50mm_Horizontal, F.Cu at (107.3, 81.8)
- added Q2: FDMC86102LZ, FDMC86102LZ:FDMC86139P, B.Cu at (115.7, 73.1)
- added R32: 1k, Resistor_SMD:R_0603_1608Metric, F.Cu at (135.5, 138.7)
- added S1: CJS-1200TB, CJS-1200TB:B-TYPE, F.Cu at (153.6, 139.2)
- added S2: CJS-1200TB, CJS-1200TB:B-TYPE, B.Cu at (140.2, 101.8)
- added S3: CJS-1200TB, CJS-1200TB:B-TYPE, B.Cu at (109.3, 76.6)
- added TP13: TestPoint, TestPoint:TestPoint_Pad_D1.0mm, F.Cu at (157.7, 142.2)
- added U5: LTC4357DCB, LTC4357IDCB#TRMPBF:SON50P300X200X80-7N-D, B.Cu at (120.7, 75.0)
- D10: value LED -> GREEN
- D11, D12: value LED -> RED
- G***: moved to B.Cu
- R26: value 0.0125 -> 0.017
- TP10: footprint TestPoint:TestPoint_Pad_D1.0mm -> TestPoint:TestPoint_Pad_D1.5mm
- TP2: footprint TestPoint:TestPoint_THTPad_D1.5mm_Drill0.7mm -> TestPoint:TestPoint_Pad_D1.5mm
- moved G*** 35.5 mm to (125.5, 114.3), turned to 90 degrees
- moved TP3 15.3 mm to (104.9, 74.7)
- moved TP2 11.7 mm to (128.6, 92.9)
- moved R3 3.93 mm to (116.6, 94.1)
- moved TP8 1.06 mm to (133.7, 140.7)
- moved C32 0.80 mm to (107.9, 91.3)
- moved D10 0.16 mm to (114.2, 139.8)
- moved D11 0.14 mm to (116.0, 139.8)
- moved D9 0.10 mm to (116.3, 137.6)
- moved R30 0.10 mm to (113.5, 137.6)
Connections:
- IC5 pad 6: /Project Architecture/Battery/BAT_P+ -> /Project Architecture/Battery/*SHDN
- J1 pad a15: /Project Architecture/Battery Charger/HVIN -> /Project Architecture/Battery Charger/HVIN_SPINE
- J1 pad a16: /Project Architecture/Battery Charger/HVIN -> /Project Architecture/Battery Charger/HVIN_SPINE
- J1 pad a2: GND -> unconnected-(J1-Pin_a2-Pada2)
- J1 pad b15: /Project Architecture/Battery Charger/HVIN -> /Project Architecture/Battery Charger/HVIN_SPINE
- J1 pad b16: /Project Architecture/Battery Charger/HVIN -> /Project Architecture/Battery Charger/HVIN_SPINE
- J1 pad b2: GND -> unconnected-(J1-Pin_b2-Padb2)
- U3 pad 1: GND -> /Project Architecture/Battery/A1
- U4 pad 1: GND -> /Project Architecture/Boost/Monitor/A1
Routing:
- net /Project Architecture/Battery/*SHDN: track 0.00 -> 74.4 mm, vias 0 -> 3
- net SDA: track 70.4 -> 133.6 mm, vias 2 -> 5
- net SCL: track 59.9 -> 115.1 mm, vias 2 -> 4
- net /Project Architecture/Battery Charger/HVIN: track 0.00 -> 33.5 mm, vias 6 -> 7
- net /Project Architecture/Battery/BAT_P+: track 19.3 -> 32.0 mm, vias 10 -> 9
- net /Project Architecture/Battery Charger/HVIN_EXT: track 0.00 -> 11.4 mm
- net /Project Architecture/Battery Charger/HVIN_SPINE: track 0.00 -> 7.76 mm, vias 0 -> 6
- net GND: track 78.0 -> 85.3 mm, vias 81 -> 138
- net /Project Architecture/Battery/A1: track 0.00 -> 7.12 mm
- net /Project Architecture/Battery Charger/BAT: track 4.18 -> 11.1 mm
- net /Project Architecture/Boost/Monitor/A1: track 0.00 -> 6.00 mm, vias 0 -> 2
- net Net-(Q2-G): track 0.00 -> 5.65 mm, vias 0 -> 2
- net Net-(D14-A): track 0.00 -> 3.81 mm
- net /Project Architecture/CHRG_OUT: track 74.6 -> 71.9 mm
- net +5V: track 81.9 -> 84.2 mm, vias 2 -> 3
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- added copper zone on B.Cu, net /Project Architecture/Battery Charger/HVIN
- added copper zone on B.Cu, net /Project Architecture/Battery Charger/HVIN_SPINE
- added copper zone on In2.Cu, net /Project Architecture/Battery Charger/HVIN_SPINE
- removed copper zone on In2.Cu, net /Project Architecture/Battery Charger/HVIN
Other:
- outline, holes or cut-outs redrawn
- board text added: "+ -"
- board text added: "0 1"
- board text added: "40"
- board text added: "41"
- board text added: "48"
- board text added: "49"
- board text added: "5V/2.5A"
- board text added: "6-24V 2.5A"
- board text added: "BAT SW"
- board text added: "Cyprien Lacassagne, 12/25"
- board text added: "HVIN: 6-36V, 2.5A OUT: VBAT+0.3, 2.5A CHRG: 1.2A, 4h NTC: [-5, 55]°C"
- board text added: "Low-Power Power Supply Unit"
- board text added: "SDA SCL GND"
- board text added: "{dblquote}On a vu souvent, rejaillir le feu de l'ancien volcan qu'on croyait trop vieux. Et quand vient le soir, pour qu'un ciel flamboie, le rouge et le noir ne s'épousent-ils pas.{dblquote}"
- board text removed: "0x40"
- board text removed: "0x41"
- board text removed: "800kHz HVIN: 6-36V, 2.5A OUT: VBAT+0.3, 2.5A CHRG: 1.2A, 3h"
- board text removed: "800kHz, 5V/2.5A"
- board text removed: "Cyprien Lacassagne, 06/12/25"
- board text removed: "Low Power Power Supply Unit"
- board text removed: "On a vu souvent, rejaillir le feu de l'ancien volcan qu'on croyait trop vieux. Et quand vient le soir, pour qu'un ciel flamboie, le rouge et le noir ne s'épousent-ils pas."
- board text removed: "VOUT"
