File: 2026_C_AV_LPSU/2026_C_AV_LPSU.kicad_sch (KiCad schematic)
At the start: 0 parts

Commit message: LPSU & TMB
Other:
- company: (none) -> EPFL Rocket Team
- title: (none) -> 2026_C_AV_LPSU "ALASTOR"
