File: 2026_C_AV_LPSU/Power - Sequencing.kicad_sch (KiCad schematic)
At the start: 0 parts

Commit message: LPSU & TMB
Other:
- company: (none) -> EPFL Rocket Team
- title: (none) -> 2026_C_AV_LPSU "ALASTOR"
Changed lines of the file:
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@@
 	(generator_version "9.0")
 	(paper "A4")
+	(title_block
+		(title "2026_C_AV_LPSU \"ALASTOR\"")
+		(date "2025-12-23")
+		(rev "1.0")
+		(company "EPFL Rocket Team")
+		(comment 1 "Cyprien Lacassagne")
+	)
 	(rectangle
 		(start 13.97 24.892)
@@
 		)
 	)
-	(text_box "Power Sequencing Diagram of your PCB here"
+	(text_box "Power Sequencing Diagram"
 		(exclude_from_sim no)
 		(at 77.47 17.78 0)
@@
 		(stroke
 			(width 0)
-			(type default)
+			(type solid)
 		)
 		(fill
