File: 2026_C_AV_LPSU/Project Architecture.kicad_sch (KiCad schematic)
At the start: 0 parts

Commit message: LPSU & TMB
Other:
- sheet Battery Charger ports: added HVIN_SPINE; removed HVIN
- sheet Spine Interface ports: added HVIN_SPINE; removed HVIN
- company: (none) -> EPFL Rocket Team
- title: (none) -> 2026_C_AV_LPSU "ALASTOR"
Changed lines of the file:
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@@
 	(generator_version "9.0")
 	(paper "A4")
+	(title_block
+		(title "2026_C_AV_LPSU \"ALASTOR\"")
+		(date "2025-12-23")
+		(rev "1.0")
+		(company "EPFL Rocket Team")
+		(comment 1 "Cyprien Lacassagne")
+	)
 	(text "Project Architecture"
 		(exclude_from_sim no)
@@
 			)
 		)
-		(pin "HVIN" input
-			(at 158.75 90.17 0)
-			(effects
-				(font
-					(size 1.27 1.27)
-				)
-				(justify right)
-			)
-		)
 		(pin "CHRG_OUT" output
 			(at 130.81 93.98 180)
@@
 				)
 				(justify left)
+			)
+		)
+		(pin "HVIN_SPINE" input
+			(at 158.75 90.17 0)
+			(effects
+				(font
+					(size 1.27 1.27)
+				)
+				(justify right)
 			)
 		)
@@
 			)
 		)
-		(pin "HVIN" output
+		(pin "HVIN_SPINE" output
 			(at 175.26 90.17 180)
 			(effects
