File: 2026_C_AV_LPSU/bat_charger.kicad_sch (KiCad schematic)
At the start: 31 parts, among them IC1 LTC4090EDJC#PBF, U1 SI2333DS-T1-E3, U2 SI2333DS-T1-E3

Commit message: LPSU & TMB
Parts:
- added D14: SBRT5A50SAF-13, SBRT5A50SAF-13:SODFL5226X110N, symbol SBRT5A50SAF-13:SBRT5A50SAF-13
- added F1: Polyfuse, 2016L260_24MR:2016L26024MR, symbol Device:Polyfuse
- added J3: Conn_01x02_Pin, TerminalBlock_Phoenix:TerminalBlock_Phoenix_PT-1,5-2-3.5-H_1x02_P3.50mm_Horizontal, symbol Connector:Conn_01x02_Pin
Connections:
- net GND: now also J3.2 (Pin_2)
- net HVIN: now also D14.1 (K)
- new net: D14.2 (A), F1.2
- new net HVIN_EXT: F1.1, J3.1 (Pin_1)
Other:
- added sheet HVIN Ideal Diode (charger_hvin_ideal_diode.kicad_sch)
- note added: "Battery charger with PowerPath control Inputs (by priority): 6V-36V DC, 3.7V Li-ion battery HVOUT/OUT: VBAT+0.3V if DC adapter present, else VBAT"
- note added: "HVIN ORing EXT: 24Vmax"
- note added: "https://www.vishay.com/docs/33011/convtabs.pdf"
- note removed: "Battery charger with PowerPath control Inputs (by priority): 6V-36V DC, 3.7V Li-ion battery HVOUT/OUT: VBAT+0.3V if DC adapter present, else VBAT Configuration: f_OSC = 800kHz -> Rt = 40.2k I_IN,MAX = 2.4A -> R_CLPROG = 422 I_CHG = 1.2A -> R_PROG = 40.2k tTIMER = 4h -> C_TIMER = 0.33uF"
- note removed: "NTC config: Charge temp. thresholds -5°C to +55°C rCOLD = 1.97k, rHOT = 13.2k https://www.vishay.com/docs/33011/convtabs.pdf"
- company: (none) -> EPFL Rocket Team
- title: (none) -> 2026_C_AV_LPSU "ALASTOR"
- moved on the sheet: C1, C2, R6
