File: 2026_C_AV_LPSU/bat_monitor.kicad_sch (KiCad schematic)
At the start: 24 parts, among them IC5 LTC4368IMS-1#PBF, Q1 FDS9926A, U3 INA228

Commit message: LPSU & TMB
Parts:
- added S1, S3: CJS-1200TB, CJS-1200TB:B-TYPE, symbol CJS-1200TB:CJS-1200TB
- added TP13: TestPoint, TestPoint:TestPoint_Pad_D1.0mm, symbol Connector:TestPoint
- D10: value LED -> GREEN
- D11: value LED -> RED
- TP2: footprint TestPoint:TestPoint_THTPad_D1.5mm_Drill0.7mm -> TestPoint:TestPoint_Pad_D1.5mm
Connections:
- net BAT_P+: now also S1.3; no longer IC5.6 (~{SHDN})
- net GND: now also S1.1, S3.1; no longer U3.1 (A1)
- net SDA: now also S3.3
- new net *SHDN: IC5.6 (~{SHDN}), S1.2, TP13.1
- new net A1: S3.2, U3.1 (A1)
Other:
- note added: "0x48"
- note added: "Address selection"
- note removed: "R_shunt = V_SHUNT_MAX / I_MAX I_MAX = 4A R_shunt = 42mOhm"
- company: (none) -> EPFL Rocket Team
- title: (none) -> 2026_C_AV_LPSU "ALASTOR"
- moved on the sheet: BT1, C10, C11, C29, C30, C32, D10, D11, D9, IC5, Q1A, Q1B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
