File: 2026_C_AV_LPSU/boost.kicad_sch (KiCad schematic)
At the start: 29 parts, among them IC3 LTC3425EUH#PBF

Commit message: LPSU & TMB
Parts:
- D12: value LED -> RED
- TP10: footprint TestPoint:TestPoint_Pad_D1.0mm -> TestPoint:TestPoint_Pad_D1.5mm
Other:
- note added: "4-Phase Boost converter"
- note removed: "4-Phase Boost converter Configuration: f_OSC = 4MHz -> Rt = 15k VOUT = 5V -> Rfb1 = 309k, Rfb2 = 100k"
- company: (none) -> EPFL Rocket Team
- title: (none) -> 2026_C_AV_LPSU "ALASTOR"
