File: 2026_C_AV_LPSU/boost_monitor.kicad_sch (KiCad schematic)
At the start: 6 parts, among them U4 INA228

Commit message: LPSU & TMB
Parts:
- added S2: CJS-1200TB, CJS-1200TB:B-TYPE, symbol CJS-1200TB:CJS-1200TB
Connections:
- net GND: now also S2.1; no longer U4.1 (A1)
- net SDA: now also S2.3
- new net A1: S2.2, U4.1 (A1)
Other:
- note added: "0x49"
- note added: "Address selection"
- note removed: "R_shunt = V_SHUNT_MAX / I_MAX V_SHUNT_MAX = 163.8mV I_MAX = 2A R_shunt = 21mOhm"
- company: (none) -> EPFL Rocket Team
- title: (none) -> 2026_C_AV_LPSU "ALASTOR"
