File: 2026_C_AV_LPSU/ideal_diode.kicad_sch (KiCad schematic)
At the start: 4 parts, among them Q3 PSMN6R4-30MLDX, U6 LTC4357DCB

Commit message: LPSU & TMB
Other:
- company: (none) -> EPFL Rocket Team
- title: (none) -> 2026_C_AV_LPSU "ALASTOR"
Changed lines of the file:
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@@
 	(generator_version "9.0")
 	(paper "A4")
+	(title_block
+		(title "2026_C_AV_LPSU \"ALASTOR\"")
+		(date "2025-12-23")
+		(rev "1.0")
+		(company "EPFL Rocket Team")
+		(comment 1 "Cyprien Lacassagne")
+	)
 	(junction
 		(at 109.22 77.47)
@@
 				)
 				(hide yes)
+			)
+		)
+		(property "Author" ""
+			(at 140.97 112.903 0)
+			(effects
+				(font
+					(size 1.27 1.27)
+				)
 			)
 		)
@@
 			)
 		)
+		(property "Author" ""
+			(at 134.112 87.757 0)
+			(effects
+				(font
+					(size 1.27 1.27)
+				)
+			)
+		)
 		(pin "1"
 		)
@@
 			)
 		)
+		(property "Author" ""
+			(at 129.54 106.553 0)
+			(effects
+				(font
+					(size 1.27 1.27)
+				)
+			)
+		)
 		(pin "1"
 		)
@@
 			)
 		)
+		(property "Author" ""
+			(at 153.67 112.903 0)
+			(effects
+				(font
+					(size 1.27 1.27)
+				)
+			)
+		)
