File: 2026_C_AV_TMB/2026_C_AV_TMB.kicad_sch (KiCad schematic)
At the start: 28 parts, among them IC1 TLV75533PDYDR, J1 DIN41612_02x16_AB, U1 RFM95W-868S2, U2 RFM95W-868S2, U3 JS4PS-1W+, U4 JS4PS-1W+

Commit message: TMB: changed SMA ref
Parts:
- AE1, AE2, AE3, AE4, AE5, AE6, AE7, AE8: footprint Connector_Coaxial:SMA_Molex_73251-2200_Horizontal -> 901-143-6RFX:9011436RFX
Changed lines of the file:
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@@
 			)
 		)
-		(property "Footprint" "Connector_Coaxial:SMA_Molex_73251-2200_Horizontal"
+		(property "Footprint" "901-143-6RFX:9011436RFX"
 			(at 109.22 110.49 0)
 			(effects
@@
 			)
 		)
-		(property "Footprint" "Connector_Coaxial:SMA_Molex_73251-2200_Horizontal"
+		(property "Footprint" "901-143-6RFX:9011436RFX"
 			(at 109.22 105.41 0)
 			(effects
@@
 			)
 		)
-		(property "Footprint" "Connector_Coaxial:SMA_Molex_73251-2200_Horizontal"
+		(property "Footprint" "901-143-6RFX:9011436RFX"
 			(at 109.22 102.87 0)
 			(effects
@@
 			)
 		)
-		(property "Footprint" "Connector_Coaxial:SMA_Molex_73251-2200_Horizontal"
+		(property "Footprint" "901-143-6RFX:9011436RFX"
 			(at 204.47 113.03 0)
 			(effects
@@
 			)
 		)
-		(property "Footprint" "Connector_Coaxial:SMA_Molex_73251-2200_Horizontal"
+		(property "Footprint" "901-143-6RFX:9011436RFX"
 			(at 204.47 102.87 0)
 			(effects
@@
 			)
 		)
-		(property "Footprint" "Connector_Coaxial:SMA_Molex_73251-2200_Horizontal"
+		(property "Footprint" "901-143-6RFX:9011436RFX"
 			(at 204.47 105.41 0)
 			(effects
@@
 			)
 		)
-		(property "Footprint" "Connector_Coaxial:SMA_Molex_73251-2200_Horizontal"
+		(property "Footprint" "901-143-6RFX:9011436RFX"
 			(at 204.47 110.49 0)
 			(effects
@@
 			)
 		)
-		(property "Footprint" "Connector_Coaxial:SMA_Molex_73251-2200_Horizontal"
+		(property "Footprint" "901-143-6RFX:9011436RFX"
 			(at 109.22 113.03 0)
 			(effects
