File: 2026_C_AV_SPINE/_autosave-spine.kicad_pcb (KiCad board)
At the start: 4 copper layers, 165 x 80 mm, 165 parts, among them IC1 LT3960EMSE#TRPBF, J1 Conn_01x02_Socket, J10 Conn_01x02_Socket, J11 DIN41612_02x16_AB, J12 SS-12800-009, J13 SS-12800-009, J14 Conn_01x02_Socket, J2 DIN41612_02x16_AB, J3 Conn_01x02_Socket, J4 SS-12800-009, J5 DIN41612_02x16_AB, J6 DIN41612_02x16_AB, J7 Conn_01x02_Socket, J8 SS-12800-009, J9 Conn_01x02_Socket, Q1 PMOS, Q10 SI7972DP-T1-GE3, Q11 SIR5607DP-T1-RE3, Q2 PMOS, Q3 PMOS, Q4 PMOS, Q5 NMOS, Q6 NMOS, Q7 NMOS, Q8 NMOS, Q9 SI7972DP-T1-GE3, U1 INA228, U2 INA228, U3 LTC4418IUF_TRPBF, U4 LM5176RHF, U5 INA228, U6 LTC4020IUHF_PBF

Commit message: added SPINE
Connections:
- J2 pad a14: +5V -> /Connectors/5Vin
- J2 pad b14: +5V -> /Connectors/5Vin
- J3 pad 1: +5V -> /Connectors/5Vin
- J3 pad 2: GND -> +5V
- J6 pad a14: +5V -> /Connectors/5Vin
- J6 pad b14: +5V -> /Connectors/5Vin
Routing:
- added copper zone on F.Cu, net /Connectors/5Vin
Changed lines of the file:
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@@
 	(net 123 "/Connectors/CAM_CAN_L")
 	(net 124 "/Connectors/CAM_CAN_H")
+	(net 125 "/Connectors/5Vin")
 	(footprint "Capacitor_SMD:C_0603_1608Metric"
 		(layer "F.Cu")
@@
 			(layers "*.Cu" "*.Mask")
 			(remove_unused_layers no)
-			(net 4 "+5V")
+			(net 125 "/Connectors/5Vin")
 			(pinfunction "Pin_a14")
 			(pintype "passive")
@@
 			(layers "*.Cu" "*.Mask")
 			(remove_unused_layers no)
-			(net 4 "+5V")
+			(net 125 "/Connectors/5Vin")
 			(pinfunction "Pin_b14")
 			(pintype "passive")
@@
 			(layers "*.Cu" "*.Mask")
 			(remove_unused_layers no)
-			(net 4 "+5V")
+			(net 125 "/Connectors/5Vin")
 			(pinfunction "Pin_a14")
 			(pintype "passive")
@@
 			(layers "*.Cu" "*.Mask")
 			(remove_unused_layers no)
-			(net 4 "+5V")
+			(net 125 "/Connectors/5Vin")
 			(pinfunction "Pin_b14")
 			(pintype "passive")
@@
 			(remove_unused_layers no)
 			(roundrect_rratio 0.25)
-			(net 4 "+5V")
+			(net 125 "/Connectors/5Vin")
 			(pinfunction "Pin_1")
 			(pintype "passive")
@@
 			(layers "*.Cu" "*.Mask")
 			(remove_unused_layers no)
-			(net 1 "GND")
+			(net 4 "+5V")
 			(pinfunction "Pin_2")
 			(pintype "passive")
@@
 	)
 	(zone
+		(net 125)
+		(net_name "/Connectors/5Vin")
+		(layer "F.Cu")
+		(hatch edge 0.5)
+		(priority 2)
+		(connect_pads yes
+			(clearance 0.4)
+		)
+		(min_thickness 0.25)
+		(filled_areas_thickness no)
+		(fill yes
+			(thermal_gap 0.3)
+			(thermal_bridge_width 0.5)
+			(smoothing chamfer)
+			(radius 0.5)
+		)
+		(polygon
+			(pts
+				(xy 101.5 90.25) (xy 101.5 92.95) (xy 148.5 92.85) (xy 148.5 89.95)
+			)
+		)
+	)
+	(zone
 		(net 1)
 		(net_name "GND")
@@
 		(polygon
 			(pts
-				(xy 42 90.1) (xy 42 92.8) (xy 148.5 92.8) (xy 148.5 89.9)
+				(xy 42 90.1) (xy 42 92.8) (xy 89 92.7) (xy 89 89.8)
 			)
 		)
