File: 2026_C_AV_SPINE/connectors.kicad_sch (KiCad schematic)
At the start: 12 parts, among them J1 Conn_01x02_Socket, J2 DIN41612_02x16_AB

Commit message: added SPINE
Parts:
- added H1, H2, H3, H4: MountingHole_Pad, MountingHole:MountingHole_3.2mm_M3_Pad, symbol Mechanical:MountingHole_Pad
- added J13: SS-12800-009, ert:STEWART_SS-12800-009, symbol SS-12800-009:SS-12800-009
- added J14: Conn_01x02_Socket, Connector_AMASS:AMASS_XT60-F_1x02_P7.20mm_Vertical, symbol Connector:Conn_01x02_Socket
- J1: footprint (none) -> Connector_AMASS:AMASS_XT60IPW-M_1x03_P7.20mm_Horizontal
- J10, J3, J7, J9: renamed from J?; footprint (none) -> Connector_AMASS:AMASS_XT60IPW-M_1x03_P7.20mm_Horizontal
- J11, J5, J6: renamed from J?; footprint (none) -> Connector_DIN:DIN41612_B2_2x16_Female_Vertical_THT
- J12, J4, J8: renamed from J?; footprint SS-12800-009:STEWART_SS-12800-009 -> ert:STEWART_SS-12800-009
- J2: footprint (none) -> Connector_DIN:DIN41612_B2_2x16_Female_Vertical_THT
Connections:
- net VIN is gone; now on net +24V: J2.a15 (Pin_a15), J2.a16 (Pin_a16), J2.b15 (Pin_b15), J2.b16 (Pin_b16), J6.a15 (Pin_a15), J6.a16 (Pin_a16), J6.b15 (Pin_b15), J6.b16 (Pin_b16)
- net +24V: now also J11.a15 (Pin_a15), J11.a16 (Pin_a16), J11.b15 (Pin_b15), J11.b16 (Pin_b16), J14.1 (Pin_1); no longer J3.1 (Pin_1)
- net +5V: now also J3.2 (Pin_2), J13.4; no longer J2.a14 (Pin_a14), J2.b14 (Pin_b14), J6.a14 (Pin_a14), J6.b14 (Pin_b14)
- net 24V_BATT: no longer J9.1 (Pin_1)
- net 24V_BATT_BCK: no longer J1.1 (Pin_1)
- net GND: now also H1.1, H2.1, H3.1, H4.1, J13.1, J13.SH1 (SHIELD), J13.SH2 (SHIELD), J14.2 (Pin_2); no longer J11.a15 (Pin_a15), J11.a16 (Pin_a16), J11.b15 (Pin_b15), J11.b16 (Pin_b16), J3.2 (Pin_2), J5.a2 (Pin_a2), J5.b2 (Pin_b2), J7.2 (Pin_2)
- net INTRANET_CAN_H: no longer J4.2
- net INTRANET_CAN_L: no longer J4.3
- net RS232_FDR_RX: now also J4.2
- net RS232_FDR_TX: now also J4.3
- new net +24V_SW: J7.2 (Pin_2)
- new net 24V_BATT_BCK_IN: J1.1 (Pin_1)
- new net 24V_BATT_IN: J9.1 (Pin_1)
- new net 5Vin: J2.a14 (Pin_a14), J2.b14 (Pin_b14), J3.1 (Pin_1), J6.a14 (Pin_a14), J6.b14 (Pin_b14)
- new net CAM_CAN_H: J13.2, J5.a2 (Pin_a2)
- new net CAM_CAN_L: J13.3, J5.b2 (Pin_b2)
