File: 2026_C_AV_SPINE/connectors.kicad_sch (KiCad schematic)
At the start: 18 parts, among them J1 Conn_01x02_Socket, J10 Conn_01x02_Socket, J11 DIN41612_02x16_AB, J12 SS-12800-009, J13 SS-12800-009, J14 Conn_01x02_Socket, J2 DIN41612_02x16_AB, J3 Conn_01x02_Socket, J4 SS-12800-009, J5 DIN41612_02x16_AB, J6 DIN41612_02x16_AB, J7 Conn_01x02_Socket, J8 SS-12800-009, J9 Conn_01x02_Socket

Commit message: spine almost finished
Parts:
- removed J12, J13, J4, J8: SS-12800-009, ert:STEWART_SS-12800-009, symbol SS-12800-009:SS-12800-009
- added H5, H6, H7, H8: MountingHole_Pad, MountingHole:MountingHole_3.2mm_M3_Pad, symbol Mechanical:MountingHole_Pad
- added J12, J13, J15: Conn_02x02, ert:SHDRRA4W55P200_2X2_665X640X630P, symbol Connector_Generic:Conn_02x02_Top_Bottom
- added J4, J8: 54-00274, ert:TENSILITY_54-00274, symbol ert:54-00274
- J14: footprint Connector_AMASS:AMASS_XT60-F_1x02_P7.20mm_Vertical -> Connector_AMASS:AMASS_XT60IPW-M_1x03_P7.20mm_Horizontal
- renumbered J9 to J1, J1 to J10, J10 to J9
Connections:
- net +24V: now also J12.3 (Pin_3), J13.3 (Pin_3), J15.3 (Pin_3); no longer J2.a15 (Pin_a15), J2.a16 (Pin_a16), J2.b15 (Pin_b15), J2.b16 (Pin_b16), J6.a15 (Pin_a15), J6.a16 (Pin_a16), J6.b15 (Pin_b15), J6.b16 (Pin_b16)
- net +5V: now also J4.3, J8.3
- net 24V_PFS: now also J2.a15 (Pin_a15), J2.a16 (Pin_a16), J2.b15 (Pin_b15), J2.b16 (Pin_b16), J6.a15 (Pin_a15), J6.a16 (Pin_a16), J6.b15 (Pin_b15), J6.b16 (Pin_b16)
- net CAM_CAN_H: now also J12.2 (Pin_2), J13.2 (Pin_2), J15.2 (Pin_2)
- net CAM_CAN_L: now also J12.4 (Pin_4), J13.4 (Pin_4), J15.4 (Pin_4)
- net GND: now also H5.1, H6.1, H7.1, H8.1, J12.1 (Pin_1), J13.1 (Pin_1), J15.1 (Pin_1), J4.1, J4.S1 (SHIELD), J4.S2 (SHIELD__1), J8.1, J8.S1 (SHIELD), J8.S2 (SHIELD__1)
- net INTRANET_CAN_H: now also J8.2
- net INTRANET_CAN_L: now also J8.4
- net RS232_FDR_RX: now also J4.2
- net RS232_FDR_TX: now also J4.4
Other:
- moved on the sheet: H1, H2, H3, H4

Commit message: Layout spine finished
Connections:
- net +24V: now also J14.2 (Pin_2); no longer J14.1 (Pin_1)
- net GND: now also J14.1 (Pin_1); no longer J14.2 (Pin_2)
Changed lines of the file:
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@@
+	(wire
+		(pts
+			(xy 142.24 127) (xy 146.05 127)
+		)
+		(stroke
+			(width 0)
+			(type default)
+		)
+	)
 	(wire
 		(pts
@@
 		(pts
 			(xy 106.68 138.43) (xy 107.95 138.43)
+		)
+		(stroke
+			(width 0)
+			(type default)
+		)
+	)
+	(wire
+		(pts
+			(xy 142.24 129.54) (xy 146.05 129.54)
 		)
 		(stroke
@@
 	)
 	(label "GND"
-		(at 146.05 129.54 180)
-		(effects
-			(font
-				(size 1.27 1.27)
-			)
-			(justify right bottom)
+		(at 142.24 127 0)
+		(effects
+			(font
+				(size 1.27 1.27)
+			)
+			(justify left bottom)
 		)
 	)
@@
 	)
 	(label "24V"
-		(at 146.05 127 180)
-		(effects
-			(font
-				(size 1.27 1.27)
-			)
-			(justify right bottom)
-		)
-	)
+		(at 142.24 129.54 0)
+		(effects
+			(font
+				(size 1.27 1.27)
+			)
+			(justify left bottom)
+		)
+	)

Commit message: updates: FC & SPINE
Parts:
- added TP5: 24V, TestPoint:TestPoint_THTPad_D3.0mm_Drill1.5mm, symbol Connector:TestPoint
- added TP6: 5V, TestPoint:TestPoint_THTPad_D3.0mm_Drill1.5mm, symbol Connector:TestPoint
Connections:
- net +24V: now also TP5.1
- net +5V: now also TP6.1
Other:
- title: FH2 - Spine -> Connectors
Changed lines of the file:
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@@
 	(paper "A4")
 	(title_block
-		(title "FH2 - Spine")
-		(date "2025-12-10")
+		(title "Connectors")
+		(date "2026-03-01")
 		(rev "v1")
 		(comment 1 "Elie Baier")
@@
 	)
 	(junction
+		(at 29.21 176.53)
+		(diameter 0)
+		(color 0 0 0 0)
+	)
+	(junction
 		(at 107.95 138.43)
 		(diameter 0)
@@
 		(color 0 0 0 0)
 	)
+	(junction
+		(at 29.21 168.91)
+		(diameter 0)
+		(color 0 0 0 0)
+	)
 	(wire
 		(pts
@@
 	(wire
 		(pts
+			(xy 29.21 168.91) (xy 30.48 168.91)
+		)
+		(stroke
+			(width 0)
+			(type default)
+		)
+	)
+	(wire
+		(pts
 			(xy 29.21 180.34) (xy 29.21 181.61)
 		)
@@
 	(wire
 		(pts
+			(xy 29.21 176.53) (xy 30.48 176.53)
+		)
+		(stroke
+			(width 0)
+			(type default)
+		)
+	)
+	(wire
+		(pts
 			(xy 182.88 115.57) (xy 195.58 115.57)
 		)
@@
 	)
 	(symbol
+		(lib_id "Connector:TestPoint")
+		(at 30.48 168.91 270)
+		(unit 1)
+		(exclude_from_sim no)
+		(in_bom yes)
+		(on_board yes)
+		(dnp no)
+		(property "Reference" "TP5"
+			(at 32.258 167.132 90)
+			(effects
+				(font
+					(size 1.27 1.27)
+				)
+				(justify left)
+			)
+		)
+		(property "Value" "24V"
+			(at 32.258 170.688 90)
+			(effects
+				(font
+					(size 1.27 1.27)
+				)
+				(justify left)
+			)
+		)
+		(property "Footprint" "TestPoint:TestPoint_THTPad_D3.0mm_Drill1.5mm"
+			(at 30.48 173.99 0)
+			(effects
+				(font
+					(size 1.27 1.27)
+				)
+				(hide yes)
+			)
+		)
+		(property "Datasheet" "~"
+			(at 30.48 173.99 0)
+			(effects
+				(font
+					(size 1.27 1.27)
+				)
+				(hide yes)
+			)
+		)
+		(property "Description" "test point"
+			(at 30.48 168.91 0)
+			(effects
+				(font
+					(size 1.27 1.27)
+				)
+				(hide yes)
+			)
+		)
+		(pin "1"
+		)
+		(instances
+			(project ""
+				(path "/9b29516b-1745-41d0-bc5f-f6cf48cfb4af/628d96ad-ccb6-491d-a37f-7a3e1150162c"
+					(reference "TP5")
+					(unit 1)
+				)
+			)
+		)
+	)
+	(symbol
 		(lib_id "Connector:Conn_01x02_Socket")
 		(at 151.13 110.49 0)
@@
 					(unit 1)
 				)
+			)
+		)
+	)
+	(symbol
+		(lib_id "Connector:TestPoint")
+		(at 30.48 176.53 270)
+		(unit 1)
+		(exclude_from_sim no)
+		(in_bom yes)
+		(on_board yes)
+		(dnp no)
+		(property "Reference" "TP6"
+			(at 32.258 174.752 90)
+			(effects
+				(font
+					(size 1.27 1.27)
+				)
+				(justify left)
+			)
+		)
+		(property "Value" "5V"
+			(at 32.258 178.308 90)
+			(effects
+				(font
+					(size 1.27 1.27)
+				)
+				(justify left)
+			)
+		)
+		(property "Footprint" "TestPoint:TestPoint_THTPad_D3.0mm_Drill1.5mm"
+			(at 30.48 181.61 0)
+			(effects
+				(font
+					(size 1.27 1.27)
+				)
+				(hide yes)
+			)
+		)
+		(property "Datasheet" "~"
+			(at 30.48 181.61 0)
+			(effects
+				(font
+					(size 1.27 1.27)
+				)
+				(hide yes)
+			)
+		)
+		(property "Description" "test point"
+			(at 30.48 176.53 0)
+			(effects
+				(font
+					(size 1.27 1.27)
+				)
+				(hide yes)
+			)
+		)
+		(pin "1"
+		)
+		(instances
+			(project "spine"
+				(path "/9b29516b-1745-41d0-bc5f-f6cf48cfb4af/628d96ad-ccb6-491d-a37f-7a3e1150162c"
+					(reference "TP6")
+					(unit 1)
+				)
