File: 2026_C_AV_SPINE/power_mgmt.kicad_sch (KiCad schematic)
At the start: 74 parts, among them Q1 PMOS, Q2 PMOS, Q3 PMOS, Q4 PMOS, Q5 NMOS, Q6 NMOS, Q7 NMOS, Q8 NMOS, U3 LTC4418IUF_TRPBF, U4 LM5176RHF

Commit message: added SPINE
Parts:
- removed D5, D6: D, symbol Device:D
- added D14, D5: LED, LED_SMD:LED_0603_1608Metric, symbol Device:LED
- C10, C11, C12, C13, C14, C15, C16, C17, C18, C19, C20, C21, C22, C23, C24, C26, C27, C28, C29, C30, C6, C7, C8, C9: footprint (none) -> Capacitor_SMD:C_0603_1608Metric
- C25: footprint (none) -> Capacitor_SMD:C_Elec_5x5.8
- C31, C32, C33, C34, C35: footprint (none) -> Capacitor_SMD:C_Elec_4x5.4
- C36, C37: footprint (none) -> Capacitor_SMD:C_Elec_6.3x7.7
- L1: footprint (none) -> Inductor_SMD:L_0603_1608Metric
- Q1, Q2, Q3, Q4: footprint (none) -> Package_SO:PowerPAK_SO-8_Single
- Q5, Q6, Q7, Q8: footprint (none) -> Package_TO_SOT_SMD:LFPAK33
- R10, R11, R12, R13, R14, R15, R16, R17, R18, R19, R20, R21, R22, R23, R24, R25, R26, R27, R28, R29, R30, R31, R32, R33, R7, R8, R9: footprint (none) -> Resistor_SMD:R_0603_1608Metric
- U3: footprint LTC4418IUF_TRPBF:QFN50P400X400X80-21N -> Package_DFN_QFN:QFN-20-1EP_4x4mm_P0.5mm_EP2.5x2.5mm_ThermalVias
- U4: footprint Package_DFN_QFN:VQFN-28-1EP_4x5mm_P0.5mm_EP2.55x3.55mm -> Package_DFN_QFN:VQFN-28-1EP_4x5mm_P0.5mm_EP2.55x3.55mm_ThermalVias
Connections:
- net QH1OUT is gone; now on net 24V_MUXOUT: C25.1, C26.2, C8.1, C9.1, Q1.1 (D), Q4.1 (D), Q7.1 (D), R26.2, R27.1, R32.2, U3.15 (VOUT)
- net 24V_NO_MON: now also C18.1, C37.2, U4.21 (BIAS)
- net GND: now also C26.1, C27.1, C28.1, C29.1, C31.1, C32.1, C33.1, C34.1, C36.1
- net QH2OUT: now also C32.2, C33.2, C34.2, C35.2
- net VALID1: now also D5.1 (K)
- net VALID2: now also D14.1 (K)
- net FB: now reaches R19.1, R20.2, U4.8 (FB)
- net OV2: now reaches R10.1, R11.2, U3.5 (OV2)
- net MODE: now reaches R25.2, U4.1 (MODE)
- net ISNS-: now reaches C20.1, R29.1, U4.10 (ISNS(-))
- net ISNS+: now reaches C20.2, R28.2, U4.11 (ISNS(+))
- net CSG: now reaches C15.1, R23.1, U4.12 (CSG)
- net CS: now reaches C15.2, R22.2, U4.13 (CS)
- net BOOT2: now reaches C22.1, U4.17 (BOOT2)
- net VCC: now reaches C17.1, U4.20 (VCC)
- net BOOT1: now reaches C21.1, U4.23 (BOOT1)
- net EN/UVLO: now reaches R32.1, R33.1, U4.26 (EN/UVLO)
- net VIN_reg: now reaches C19.1, R27.2, U4.27 (VIN)
- net VISNS: now reaches R26.1, U4.28 (VISNS)
- net RT: now reaches R18.2, U4.3 (RT/SYNC)
- net SLOPE: now reaches C12.1, U4.4 (SLOPE)
- net SS: now reaches C16.2, U4.5 (SS)
- net at R17.1: now also D14.2 (A)
- net at R16.1: now also D5.2 (A)
- net 24V_MUXOUT: now reaches C30.2
- net 24V_MUXOUT: now also C27.2, C28.2, C29.2; no longer C29.1
- net TMR: now reaches C13.1, U3.1 (TMR)
- net EN: now reaches C14.2, U3.10 (INTVCC), U3.18 (EN), U3.19 (~{SHDN})
- net UV1: now reaches R8.1, R9.2, U3.2 (UV1)
- net HYS: now reaches R15.1, U3.20 (HYS)
- net OV1: now reaches R7.1, R8.2, U3.3 (OV1)
- net UV2: now reaches R11.1, R12.2, U3.4 (UV2)
Other:
- moved on the sheet: C26, C27, C28, C29, C30, C31, C32, C33, C34, C35, C36, C37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
