File: 2026_C_AV_SPINE/power_mon.kicad_sch (KiCad schematic)
At the start: 21 parts, among them IC1 LT3960EMSE#TRPBF, U1 INA228, U2 INA228, U5 INA228

Commit message: added SPINE
Parts:
- removed D1, D2, D7: D, symbol Device:D
- added D1, D2, D6: LED, LED_SMD:LED_0603_1608Metric, symbol Device:LED
- C1, C2, C3, C38, C4, C5: footprint (none) -> Capacitor_SMD:C_0603_1608Metric
- IC1: footprint SOP50P490X110-11N -> ert:SOP50P490X110-11N
- R1, R2, R3, R34, R35, R4, R5, R6: footprint (none) -> Resistor_SMD:R_0603_1608Metric
Connections:
- net 24V_BATT: no longer R2.1, U2.10 (Vin+), U2.8 (Vbus)
- net 24V_BATT_BCK: no longer R34.1, U5.10 (Vin+), U5.8 (Vbus)
- net at U2.3 (~{Alert}): now also D2.1 (K)
- net at R4.1: now also D2.2 (A)
- net at R35.1: now also D1.2 (A)
- net at U1.3 (~{Alert}): now also D6.1 (K)
- net at R3.1: now also D6.2 (A)
- net at U5.3 (~{Alert}): now also D1.1 (K)
- net +24V renamed +24V_SW
- new net 24V_BATT_BCK_IN: R34.1, U5.10 (Vin+), U5.8 (Vbus)
- new net 24V_BATT_IN: R2.1, U2.10 (Vin+), U2.8 (Vbus)
