File: 2026_C_AV_SPINE/power_mon.kicad_sch (KiCad schematic)
At the start: 21 parts, among them IC1 LT3960EMSE#TRPBF, U1 INA228, U2 INA228, U5 INA228

Commit message: spine almost finished
Parts:
- R1, R2, R34: value 2m -> 10m; footprint Resistor_SMD:R_0603_1608Metric -> Resistor_SMD:R_2512_6332Metric; Mouser (none) -> https://www.mouser.ch/ProductDetail/Vishay-Dale/WSLP2512R01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
Connections:
- net 24V_NO_MON renamed 24V_OUT_REG
Other:
- moved on the sheet: C1, C2, C38, D1, D2, D6, R1, R3, R35, R4, U1, U2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
