File: 2026_C_AV_SPINE/power.kicad_sch (KiCad schematic)
At the start: 0 parts

Commit message: spine almost finished
Other:
- sheet Charger ports: added none; removed 24V_OUT_CHARGER
- sheet Management ports: added none; removed 24V_NO_MON, 24V_OUT_CHARGER
- sheet Monitoring ports: added none; removed 24V_NO_MON
Changed lines of the file:
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@@
 		(comment 1 "Elie Baier")
-	)
-	(wire
-		(pts
-			(xy 303.53 86.36) (xy 303.53 121.92)
-		)
-		(stroke
-			(width 0)
-			(type default)
-		)
-	)
-	(wire
-		(pts
-			(xy 304.8 86.36) (xy 303.53 86.36)
-		)
-		(stroke
-			(width 0)
-			(type default)
-		)
-	)
-	(wire
-		(pts
-			(xy 302.26 83.82) (xy 302.26 104.14)
-		)
-		(stroke
-			(width 0)
-			(type default)
-		)
-	)
-	(wire
-		(pts
-			(xy 302.26 104.14) (xy 304.8 104.14)
-		)
-		(stroke
-			(width 0)
-			(type default)
-		)
-	)
-	(wire
-		(pts
-			(xy 303.53 121.92) (xy 304.8 121.92)
-		)
-		(stroke
-			(width 0)
-			(type default)
-		)
-	)
-	(wire
-		(pts
-			(xy 304.8 83.82) (xy 302.26 83.82)
-		)
-		(stroke
-			(width 0)
-			(type default)
-		)
 	)
 	(sheet
@@
 				)
 				(justify left top)
-			)
-		)
-		(pin "24V_NO_MON" input
-			(at 304.8 104.14 180)
-			(effects
-				(font
-					(size 1.27 1.27)
-				)
-				(justify left)
 			)
 		)
@@
 			)
 		)
-		(pin "24V_NO_MON" input
-			(at 304.8 83.82 180)
-			(effects
-				(font
-					(size 1.27 1.27)
-				)
-				(justify left)
-			)
-		)
-		(pin "24V_OUT_CHARGER" input
-			(at 304.8 86.36 180)
-			(effects
-				(font
-					(size 1.27 1.27)
-				)
-				(justify left)
-			)
-		)
 		(instances
 			(project "spine"
@@
 			)
 		)
-		(pin "24V_OUT_CHARGER" input
-			(at 304.8 121.92 180)
-			(effects
-				(font
-					(size 1.27 1.27)
-				)
-				(justify left)
-			)
-		)
