File: 2026_C_AV_SPINE/spine.kicad_pcb (KiCad board)
At the start: 4 copper layers, 165 x 80 mm, 181 parts, among them IC1 LT3960EMSE#TRPBF, J1 Conn_01x02_Socket, J10 Conn_01x02_Socket, J11 DIN41612_02x16_AB, J12 Conn_02x02, J13 Conn_02x02, J14 Conn_01x02_Socket, J15 Conn_02x02, J2 DIN41612_02x16_AB, J3 Conn_01x02_Socket, J4 54-00274, J5 DIN41612_02x16_AB, J6 DIN41612_02x16_AB, J7 Conn_01x02_Socket, J8 54-00274, J9 Conn_01x02_Socket, Q1 STL42P6LLF6, Q10 STL42P6LLF6, Q11 STL42P6LLF6, Q12 STL36DN6F7, Q13 STL42P6LLF6, Q2 STL42P6LLF6, Q5 STL8N10F7, Q6 STL8N10F7, Q7 STL8N10F7, Q8 STL8N10F7, Q9 STL36DN6F7, U1 INA228, U2 INA228, U3 LTC4418IUF_TRPBF, U4 LM5176RHF, U5 INA228, U6 LTC4020IUHF_PBF

Commit message: Layout spine finished
Parts:
- added TP1: SHND, TestPoint:TestPoint_Pad_D2.0mm, F.Cu at (234.6, 128.3)
- added TP2: VOUT_CHARGER, TestPoint:TestPoint_Pad_D2.0mm, F.Cu at (221.9, 104.5)
- added TP3: VIN_CHARGER, TestPoint:TestPoint_Pad_D2.0mm, F.Cu at (154.7, 61.8)
- added TP4: VBAT, TestPoint:TestPoint_Pad_D2.0mm, F.Cu at (214.0, 122.5)
- H5, H6, H7, H8: value MountingHole_3.2mm_M3_DIN965_Pad -> MountingHole_Pad; footprint MountingHole:MountingHole_3.2mm_M3_DIN965_Pad -> MountingHole:MountingHole_3.2mm_M3_Pad
- renumbered J3 to J14, J14 to J3
Connections:
- J14 pad 1: /Connectors/5Vin -> GND
- J14 pad 2: +5V -> +24V
- J3 pad 1: +24V -> /Connectors/5Vin
- J3 pad 2: GND -> +5V
Routing:
- net +24V: track 165.4 -> 213.2 mm
- net +5V: track 361.0 -> 392.5 mm
- net GND: track 139.4 -> 144.4 mm, vias 67 -> 66
- net /Power/Management/24V_MUXOUT: track 39.0 -> 43.4 mm
- net /Power/Management/VALID2: track 89.4 -> 87.0 mm, vias 0 -> 2
- net /Power/Management/VALID1: track 93.1 -> 91.0 mm, vias 0 -> 2
- net /Connectors/5Vin: track 60.3 -> 62.0 mm
- net /Power/Management/VCC: track 44.5 -> 45.7 mm
- net /Power/Management/RT: track 10.2 -> 9.46 mm
- net 24V_OUT_REG: track 70.4 -> 71.0 mm
- net +24V_SW: track 24.0 -> 24.6 mm
- net /Power/Management/SLOPE: track 9.63 -> 9.07 mm
- net /Power/Management/SS: track 9.71 -> 9.18 mm
- added copper zone on B.Cu, net +24V
- added copper zone on F.Cu, net +24V_SW
