File: 2026_C_AV_SPINE/spine.kicad_pcb (KiCad board)
At the start: 4 copper layers, 165 x 80 mm, 185 parts, among them IC1 LT3960EMSE#TRPBF, J1 Conn_01x02_Socket, J10 Conn_01x02_Socket, J11 DIN41612_02x16_AB, J12 Conn_02x02, J13 Conn_02x02, J14 Conn_01x02_Socket, J15 Conn_02x02, J2 DIN41612_02x16_AB, J3 Conn_01x02_Socket, J4 54-00274, J5 DIN41612_02x16_AB, J6 DIN41612_02x16_AB, J7 Conn_01x02_Socket, J8 54-00274, J9 Conn_01x02_Socket, Q1 STL42P6LLF6, Q10 STL42P6LLF6, Q11 STL42P6LLF6, Q12 STL36DN6F7, Q13 STL42P6LLF6, Q2 STL42P6LLF6, Q5 STL8N10F7, Q6 STL8N10F7, Q7 STL8N10F7, Q8 STL8N10F7, Q9 STL36DN6F7, U1 INA228, U2 INA228, U3 LTC4418IUF_TRPBF, U4 LM5176RHF, U5 INA228, U6 LTC4020IUHF_PBF

Commit message: updates: FC & SPINE
Parts:
- added G***: LOGO, LOGO, F.Cu at (210.8, 126.3)
- added G***: LOGO, LOGO, F.Cu at (234.2, 127.0)
- added G***: LOGO, LOGO, B.Cu at (227.1, 117.6)
- added G***: LOGO, LOGO, B.Cu at (218.6, 129.2)
- added G***: LOGO, LOGO, B.Cu at (201.7, 129.2)
- added G***: LOGO, LOGO, F.Cu at (77.0, 82.7)
- added G***: LOGO, LOGO, F.Cu at (77.0, 114.7)
- added G***: LOGO, LOGO, F.Cu at (227.5, 134.8)
- added G***: LOGO, LOGO, F.Cu at (192.5, 60.2)
- added G***: LOGO, LOGO, F.Cu at (80.5, 72.7)
- added G***: LOGO, LOGO, F.Cu at (225.4, 109.8)
- added G***: LOGO, LOGO, F.Cu at (194.0, 126.5)
- added R30: 38k, Resistor_SMD:R_0603_1608Metric, B.Cu at (230.1, 69.0)
- added R57: 10k, Resistor_SMD:R_0603_1608Metric, B.Cu at (233.3, 69.0)
- added TP5: 24V, TestPoint:TestPoint_THTPad_D3.0mm_Drill1.5mm, F.Cu at (151.3, 135.9)
- added TP6: 5V, TestPoint:TestPoint_THTPad_D3.0mm_Drill1.5mm, F.Cu at (157.3, 135.9)
- added TP7: VOUT_REG, TestPoint:TestPoint_Pad_D2.0mm, F.Cu at (189.4, 68.7)
- added TP8: VOUT_MUX, TestPoint:TestPoint_Pad_D1.5mm, F.Cu at (215.2, 87.6)
- L1: footprint Inductor_SMD:L_10.4x10.4_H4.8 -> Inductor_SMD:L_12x12mm_H6mm
- R16, R17: moved to F.Cu
- moved D5 85.6 mm to (227.6, 132.3), turned to 90 degrees
- moved R16 83.0 mm to (227.6, 129.2)
- moved D14 81.3 mm to (231.7, 126.8), turned to 180 degrees
- moved R17 79.4 mm to (228.5, 126.8), turned to 180 degrees
- moved G*** 5.74 mm to (88.8, 70.9)
- moved D6 4.30 mm to (187.0, 61.4)
- moved R3 4.30 mm to (187.0, 61.4)
- moved G*** 2.67 mm to (111.8, 70.9)
- moved C36 1.68 mm to (193.8, 92.6)
- moved L1 1.43 mm to (206.6, 90.3)
- moved TP1 0.82 mm to (234.4, 129.1)
- moved TP4 0.80 mm to (214.0, 123.3)
- moved Q13 0.73 mm to (217.8, 99.3)
- moved Q2 0.73 mm to (217.8, 91.8)
- moved TP2 0.55 mm to (221.9, 104.0)
Connections:
- R16 pad 2: +5V -> /Power/Management/5V_LED
- R17 pad 2: +5V -> /Power/Management/5V_LED
Routing:
- net /Power/Management/5V_LED: track 0.00 -> 64.6 mm, vias 0 -> 2
- net /Power/Charger/SHDN: track 20.4 -> 54.6 mm, vias 2 -> 3
- net +5V: track 392.5 -> 414.2 mm, vias 5 -> 4
- net +24V: track 213.2 -> 231.8 mm
- net 24V_PFS: track 151.2 -> 169.4 mm, vias 7 -> 8
- net /Power/Management/VALID2: track 87.0 -> 74.3 mm
- net GND: track 144.4 -> 135.4 mm, vias 66 -> 68
- net /Power/Management/VALID1: track 91.0 -> 82.6 mm
- net +24V_SW: track 24.6 -> 30.7 mm
- net I2C_MON_SCLL: track 106.4 -> 100.9 mm
- net /Power/Management/VCC: track 45.7 -> 40.6 mm
- net I2C_MON_SCLH: track 105.4 -> 100.8 mm
- net Net-(D6-K): track 13.1 -> 9.85 mm
- net /Power/Charger/BST1: track 49.3 -> 51.5 mm
- net /Power/Management/24V_MUXOUT: track 43.4 -> 41.2 mm, vias 15 -> 12
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Other:
- board text added: "-"
- board text added: "24V BATT"
- board text added: "24V OUT"
- board text added: "24V SWITCH"
- board text added: "24V_PFS"
- board text added: "5V"
- board text added: "5V SWITCH"
- board text added: "CAMERA"
- board text added: "CHARGER"
- board text added: "Charger: LTC4020 Max charge current: 4A Input PFS: 22-26V"
- board text added: "FDR"
- board text added: "MUX"
- board text added: "PRC"
- board text added: "Power MUX: LTC4418 Priority: main battery Switching voltage: 17V"
- board text added: "REGULATOR"
- board text added: "Regulator: LM2176 Output: 24.75V Current: 17.5A"
- board text added: "SHDN"
- board text added: "VOUT_CH"
- board text added: "VOUT_MUX"
- board text added: "VOUT_REG"
- board text added: "YGGDRASIL"
- board text added: "{dblquote}We may say that a system is a complex of interacting elements.{dblquote} - Ludwig von Bertalanffy"
