File: 2026_C_AV_SPINE/power_charger.kicad_sch (KiCad schematic)
At the start: 54 parts

Commit message: added SPINE
Parts:
- removed D? (x2): D, symbol Device:D
- added D12, D7: LED, LED_SMD:LED_0603_1608Metric, symbol Device:LED
- C39, C41, C42, C43, C44, C45, C46, C47, C48, C49, C50, C52, C53, C54, C56, C57, C58, C59, C60: renamed from C?; footprint (none) -> Capacitor_SMD:C_0603_1608Metric
- C40: renamed from C?; footprint (none) -> Capacitor_SMD:C_Elec_4x5.4
- C51, C55: renamed from C?; footprint (none) -> Capacitor_SMD:C_Elec_5x5.4
- D10, D11: renamed from D?; footprint (none) -> Diode_SMD:D_SMB
- D8, D9: renamed from D?; footprint (none) -> Diode_SMD:D_SOD-123
- L2: renamed from L?; footprint (none) -> Inductor_SMD:L_0603_1608Metric
- Q10, Q9: renamed from Q?; footprint SI7288DPT1GE3 -> Package_SO:PowerPAK_SO-8_Dual
- Q11: renamed from Q?; footprint SI7852ADPT1GE3 -> Package_SO:PowerPAK_SO-8_Dual
- R36, R37, R38, R39, R40, R41, R42, R43, R44, R45, R46, R47, R48, R49, R50, R51, R52, R53, R54, R55, R56: renamed from R?; footprint (none) -> Resistor_SMD:R_0603_1608Metric
- U6: renamed from U?; footprint LTC4020IUHF_PBF:QFN-38_UHF -> Package_DFN_QFN:WQFN-38-1EP_5x7mm_P0.5mm_EP3.15x5.15mm_ThermalVias
Connections:
- net SENSGND is gone; now on net GND: C48.2, R43.2, U6.4 (SENSGND)
- net S_4 is gone; now on net GND: Q10.3 (S2)
- net 24V_OUT_CHARGER: now also C54.1, C55.2, C56.1, C57.1
- net 24V_PFS: now also C60.1
- net GND: now also C50.2, C51.1, C54.2, C56.2, C58.2
- net STAT1: now also D7.1 (K)
- net STAT2: now also D12.1 (K)
- net at R55.1: now also D7.2 (A)
- net CSN: now reaches C49.1, R50.1, U6.22 (CSN)
- net at R56.1: now also D12.2 (A)
- net VFBMIN: now reaches R49.2, R51.1, U6.19 (VFBMIN)
- net VBG: now reaches R45.1, R49.1, R52.1, U6.18 (FBG)
- net VFB: now reaches R45.2, R47.1, U6.17 (VFB)
Other:
- moved on the sheet: C48, C50, C51, C54, C55, C56, C57, C58, C59, C60, R43

Commit message: spine almost finished
Parts:
- removed C46: 1u, Capacitor_SMD:C_0603_1608Metric, symbol Device:C
- removed C51, C55: 56u, Capacitor_SMD:C_Elec_5x5.4, symbol Device:C
- removed D10, D11: MBRS360, Diode_SMD:D_SMB, symbol Device:D
- removed D8, D9: SBR0560S1, Diode_SMD:D_SOD-123, symbol Device:D
- removed Q10, Q9: SI7972DP-T1-GE3, Package_SO:PowerPAK_SO-8_Dual, symbol SI7972DP-T1-GE3:SI7972DP-T1-GE3
- removed Q11: SIR5607DP-T1-RE3, Package_SO:PowerPAK_SO-8_Dual, symbol SIR5607DP-T1-RE3:SIR5607DP-T1-RE3
- removed R38: 100k, Resistor_SMD:R_0603_1608Metric, symbol Device:R
- added C46, C51, C55, C61: 47u, Capacitor_SMD:CP_Elec_6.3x9.9, symbol Device:C_Polarized_US
- added D10: SZBZX84C6V2LT3G, Package_TO_SOT_SMD:SOT-23-3, symbol Device:D_Zener
- added D11, D8, D9: CMSH3-40MA, Diode_SMD:D_SMA, symbol Device:D_Schottky
- added Q10: STL42P6LLF6, ert:STL42P6LLF6, symbol ert:STL42P6LLF6
- added Q12, Q9: STL36DN6F7, ert:STL36DN6F7, symbol ert:STL36DN6F7
- added R38: 50k, Resistor_SMD:R_0603_1608Metric, symbol Device:R_Small
- added TP1: SHND, TestPoint:TestPoint_THTPad_D2.0mm_Drill1.0mm, symbol Connector:TestPoint
- added TP2: VOUT_CHARGER, TestPoint:TestPoint_THTPad_D2.0mm_Drill1.0mm, symbol Connector:TestPoint
- added TP3: VIN_CHARGER, TestPoint:TestPoint_THTPad_D2.0mm_Drill1.0mm, symbol Connector:TestPoint
- added TP4: VBAT, TestPoint:TestPoint_THTPad_D2.0mm_Drill1.0mm, symbol Connector:TestPoint
- added TP5: FBG, TestPoint:TestPoint_THTPad_D2.0mm_Drill1.0mm, symbol Connector:TestPoint
- C44: value 680p -> 10n
- C48: value 0.033u -> 0.33u; name (none) -> CSENSB
- L2: value 15u -> 1u; footprint Inductor_SMD:L_0603_1608Metric -> Inductor_SMD:L_10.4x10.4_H4.8; Mouser (none) -> https://www.mouser.ch/ProductDetail/KEMET/MPX1D1040L1R0?qs=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; no (none) -> MPX1D1040L1R0
- R37: value 5m -> 3m; footprint Resistor_SMD:R_0603_1608Metric -> Resistor_SMD:R_1210_3225Metric; Mouser (none) -> https://www.mouser.ch/ProductDetail/ROHM-Semiconductor/PMR2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; name (none) -> RSENSA
- R43: value 5m -> 3m; footprint Resistor_SMD:R_0603_1608Metric -> Resistor_SMD:R_1210_3225Metric; Mouser (none) -> https://www.mouser.ch/ProductDetail/ROHM-Semiconductor/PMR2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; name (none) -> RSENSB
- R48: value 10m -> 12m; footprint Resistor_SMD:R_0603_1608Metric -> Resistor_SMD:R_2512_6332Metric; name (none) -> RSC
- R53: value 82k5 -> 80k
- R54: value 20k -> 47k5
- U6: footprint Package_DFN_QFN:WQFN-38-1EP_5x7mm_P0.5mm_EP3.15x5.15mm_ThermalVias -> Package_DFN_QFN:QFN-38-1EP_4x6mm_P0.4mm_EP2.65x4.65mm_ThermalVias
Connections:
- net 24V_BATT: now also Q10.5 (D_1), Q10.6 (D_2), Q10.7 (D_3), Q10.8 (D_4), Q10.9 (D_5), TP4.1
- net 24V_PFS: now also C55.1, C61.1, TP3.1
- net BST1: now also D9.1 (K)
- net BST2: now also D10.1 (K), D8.1 (K)
- net GND: now also C46.2, C51.2, C55.2, C61.2, Q9.1 (S2), R38.1
- net INTVCC: now also D8.2 (A), D9.2 (A)
- net SHDN: now also TP1.1
- net S_5: now also Q10.1 (S_1), Q10.2 (S_2), Q10.3 (S_3)
- net TIMER: now reaches C45.1, U6.14 (TIMER)
- net VC: now reaches C42.1, R40.2, U6.28 (VC)
- net RT: now reaches U6.8 (RT)
- net RT: now also R38.2
- net RNG/SS: now reaches C47.1, R42.1, U6.15 (RNG/SS)
- net ITH: now reaches R41.2, U6.27 (ITH)
- net 24V_OUT_CHARGER renamed VOUT_CHARG
- net VOUT_CHARG: now also C46.1, C51.1, D11.1 (K), Q9.10 (D1_3), Q9.5 (D1_1), Q9.6 (D1_2), TP2.1
- net D_1 renamed SENSTOP
- net SENSTOP: now also Q12.10 (D1_3), Q12.5 (D1_1), Q12.6 (D1_2)
- net D_2 renamed SW1
- net SW1: now also Q12.3 (S1), Q12.7 (D2_1), Q12.8 (D2_2), Q12.9 (D2_3)
- net D_4 renamed SW2
- net SW2: now also D10.2 (A), D11.2 (A), Q9.3 (S1), Q9.7 (D2_1), Q9.8 (D2_2), Q9.9 (D2_3)
- net G_1 renamed TG1
- net TG1: now also Q12.4 (G1)
- net G_2 renamed BG1
- net BG1: now also Q12.2 (G2)
- net G_3 renamed TG2
- net TG2: now also Q9.4 (G1)
- net G_4 renamed BG2
- net BG2: now also Q9.2 (G2)
- net G_5 renamed BGATE
- net BGATE: now also Q10.4 (G)
- net S_2 renamed SENSBOT
- net SENSBOT: now also Q12.1 (S2)
- net VBG renamed FBG
- net FBG: now also TP5.1
Other:
- note added: "Kelvin sens - 1210"
- note added: "Notes: - BAT. Vfloat (RFB) is given by 2.5*(1+(R47/R45)) => 2.5*(1+(90.9/10)) = 25.225 (vs. 25.20 in 2026_C_SE_PTS) - VOUT min. (RMIN) given by 2.125*(1+(R51/R49)) => 2.125*(1+(${/9b29516b-1745-41d0-bc5f-f6cf48cfb4af/19f231c9-3ea2-4c72-8861-e175feaab368/ec5f26d7-fdd0-48e9-b0a5-29a04a3f71db/77b7c961-89a9-43a2-9149-ac2a1fc6824a:VALUE}/${/9b29516b-1745-41d0-bc5f-f6cf48cfb4af/19f231c9-3ea2-4c72-8861-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"
- note removed: "Notes: - BAT. Vfloat (RFB) is given by 2.5*(1+(R5/R4)) => 2.5*(1+(90.9/10)) = 25.225 (vs. 25.20 in 2026_C_SE_PTS) - VOUT min. (RMIN) given by 2.125*(1+(R8/R9)) => 2.125*(1+(94.2/10)) = 22.14V - VOUT max. (RMAX) given by 2.75*(1+(R20/R21)) => 2.75*(1+(82/10)) = 25.3V - BAT. max. I (input) set to 5A max. => 0.05/R14 = 0.05/0.01 = 5A - VIN max. I set to 10A max. (5A BAT. + 5A load) => 0.05/(R3 = R10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"
- moved on the sheet: C39, C40, C41, C42, C43, C44, C45, C47, C48, C49, C50, C52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

Commit message: updates: FC & SPINE
Parts:
- removed TP5: FBG, TestPoint:TestPoint_THTPad_D2.0mm_Drill1.0mm, symbol Connector:TestPoint
- TP1, TP2, TP3, TP4: footprint TestPoint:TestPoint_THTPad_D2.0mm_Drill1.0mm -> TestPoint:TestPoint_Pad_D2.0mm
Other:
- moved on the sheet: C48, R43
