File: 2026_C_AV_FDR/2026_C_AV_FDR.kicad_pcb (KiCad board)
At the start: 4 copper layers, 50 x 40 mm, 100 parts, among them IC1 MIC94060YMT-TR, J1 microSD_holder, J2 USB_C_Receptacle, J3 SPINE_in, J4 Conn_01x08_Pin, Q2 IRLML2502, SW1 SW_Omron_B3U, SW3 SW_SPDT, SW4 SW_SPDT, U1 RGBLED_1, U2 TPS2116DRL, U3 MCP1727-3302xSN, U4 STM32L476RGTx, U5 INA228, U6 MAX3226, U8 USBLC6-2P6, U9 TMP1075DSG

Commit message: spine almost finished
Parts:
- added G***: LOGO, LOGO, F.Cu at (134.4, 84.4)
