File: 2026_C_AV_FDR/Block Diagram.kicad_sch (KiCad schematic)
At the start: 0 parts

Commit message: spine almost finished
Other:
- title: PROMETHEUS -> Propultion Computer
Changed lines of the file:
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@@
 	(paper "A3")
 	(title_block
-		(title "PROMETHEUS")
-		(date "2025-11-19")
+		(title "Propultion Computer")
+		(date "2026-02-19")
 		(company "EPFL Rocket Team")
 		(comment 1 "Julian Ruiz Rodriguez")
