File: 2026_C_AV_PC_V1/2026_C_AV_PC_V1.kicad_pcb (KiCad board)
At the start: 4 copper layers, 115 x 50 mm, 272 parts, among them IC1 INA228AIDGSR, IC2 FAN3227TMX, IC3 FAN3227TMX, IC4 MCP1642D-50I_MS, IC5 FAN3227TMX, IC6 ADP1610ARMZ-R7, IC7 FDC1004DGSR, IC8 LTC3878EGN#PBF, IC9 TPS25221DRVR, J1 Sens2, J10 microSD_holder, J11 Kulite, J12 Me-b, J13 MO-bc, J14 IGNITER, J15 SPINE_out, J16 FLS, J17 Sens5, J18 Conn_01x05_Pin, J19 USB_B_Mini, J2 PT1000-2, J20 Me-b, J21 MO-bc, J22 24Vout, J23 Sens1, J24 PT1000-1, J25 PT1000-4, J26 Ball_valve, J27 Conn_01x05_Pin, J3 PT1000-3, J4 Sens3, J5 Sens4, J6 EXT, J7 USB_B_Mini, J8 24Vin, J9 SPINE_in, Q1 IRLML2502, Q2 STS5DNF60L, Q3 BSC093N04LSGATMA1, Q4 STS5DNF60L, Q5 BSC093N04LSGATMA1, SW2 SW_SPDT, SW3 SW_Omron_B3U, U1 MCP602, U10 TPS2116DRL, U11 MCP602, U12 USBLC6-2P6, U13 USBLC6-2P6, U2 PCA9547PW, U3 INA128, U4 LMT85DCK, U5 MCP1727-3302xSN, U6 MCP2542FDxMF, U7 RGBLED_1, U8 RGBLED_2, U9 STM32H743VIT6, Y1 16MHz

Commit message: spine almost finished
Routing:
- net +24V: vias 19 -> 18
- net GND: vias 148 -> 155
